File: LampBoxV0.31-THT.brd (EAGLE design)
At the start: 100 x 20 mm, 21 parts

Commit message: updated pcb files and readme
Parts:
- added LOGO1: OSHW-LOGOMINI, SparkFun-Aesthetics:OSHW-LOGO-MINI
- F1: value PTCPTH -> LITTELFUSE_RXEF050LITTELFUSE_RXEF050_0_0; device movuino:PTC -> movuino:LITTELFUSE_RXEF050_0
- moved C1 0.40 mm to (92.0, 14.3)
- moved F1 0.40 mm to (15.1, 15.8)
Connections:
- net +5V: now also F1.2; no longer F1.P$2
- net VIN: now also F1.1; no longer F1.P$1
Routing:
- net VIN: track 11.3 -> 12.0 mm
Other:
- board text added: "V0.31-THT"
- board text removed: "V0.3-THT"
